File: PCB/CrowMiniMk2.sch (KiCad schematic (older format))
At the start: 21 parts, among them J1 AVR-ISP-6, SW1 SW_Push, U1 ATmega32U4-AU, U2 PRTR5V0U2X, X1 XTAL

Commit message: PCB Manufacturing
Parts:
- added H1, H2, H3, H4, H5: MountingHole, MountingHole:MountingHole_2.2mm_M2_Pad, symbol Mechanical:MountingHole
Other:
- note added: "Holes"
Changed lines of the file:
@@
 $EndComp
 Connection ~ 6700 3200
+$Comp
+L Mechanical:MountingHole H1
+U 1 1 61538AC8
+P 8500 5000
+F 0 "H1" H 8600 5046 50  0000 L CNN
+F 1 "MountingHole" H 8600 4955 50  0000 L CNN
+F 2 "MountingHole:MountingHole_2.2mm_M2_Pad" H 8500 5000 50  0001 C CNN
+F 3 "~" H 8500 5000 50  0001 C CNN
+	1    8500 5000
+	1    0    0    -1
+$EndComp
+$Comp
+L Mechanical:MountingHole H2
+U 1 1 61570DD6
+P 8500 5200
+F 0 "H2" H 8600 5246 50  0000 L CNN
+F 1 "MountingHole" H 8600 5155 50  0000 L CNN
+F 2 "MountingHole:MountingHole_2.2mm_M2_Pad" H 8500 5200 50  0001 C CNN
+F 3 "~" H 8500 5200 50  0001 C CNN
+	1    8500 5200
+	1    0    0    -1
+$EndComp
+$Comp
+L Mechanical:MountingHole H3
+U 1 1 615711C1
+P 8500 5400
+F 0 "H3" H 8600 5446 50  0000 L CNN
+F 1 "MountingHole" H 8600 5355 50  0000 L CNN
+F 2 "MountingHole:MountingHole_2.2mm_M2_Pad" H 8500 5400 50  0001 C CNN
+F 3 "~" H 8500 5400 50  0001 C CNN
+	1    8500 5400
+	1    0    0    -1
+$EndComp
+$Comp
+L Mechanical:MountingHole H4
+U 1 1 615713C2
+P 8500 5600
+F 0 "H4" H 8600 5646 50  0000 L CNN
+F 1 "MountingHole" H 8600 5555 50  0000 L CNN
+F 2 "MountingHole:MountingHole_2.2mm_M2_Pad" H 8500 5600 50  0001 C CNN
+F 3 "~" H 8500 5600 50  0001 C CNN
+	1    8500 5600
+	1    0    0    -1
+$EndComp
+$Comp
+L Mechanical:MountingHole H5
+U 1 1 615715A4
+P 8500 5800
+F 0 "H5" H 8600 5846 50  0000 L CNN
+F 1 "MountingHole" H 8600 5755 50  0000 L CNN
+F 2 "MountingHole:MountingHole_2.2mm_M2_Pad" H 8500 5800 50  0001 C CNN
+F 3 "~" H 8500 5800 50  0001 C CNN
+	1    8500 5800
+	1    0    0    -1
+$EndComp
+Wire Notes Line
+	9350 4800 9350 6000
+Wire Notes Line
+	9350 6000 8200 6000
+Wire Notes Line
+	8200 6000 8200 4800
+Wire Notes Line
+	8200 4800 9350 4800
+Text Notes 8150 4800 0    197  ~ 0
+Holes
 $EndSCHEMATC

Commit message: Save1.2.2
Parts:
- C1, C2, C3: footprint Capacitor_SMD:C_0805_2012Metric_Pad1.15x1.40mm_HandSolder -> Capacitor_SMD:C_0805_2012Metric; LCSC (none) -> C62912
- C5: footprint Capacitor_SMD:C_0805_2012Metric_Pad1.15x1.40mm_HandSolder -> Capacitor_SMD:C_0805_2012Metric; LCSC (none) -> C95841
- C6: footprint Capacitor_SMD:C_0805_2012Metric_Pad1.15x1.40mm_HandSolder -> Capacitor_SMD:C_0805_2012Metric; LCSC (none) -> C116352
- C7, C8: footprint Capacitor_SMD:C_0805_2012Metric_Pad1.15x1.40mm_HandSolder -> Capacitor_SMD:C_0805_2012Metric; LCSC (none) -> C1804
- F1: footprint Fuse:Fuse_1206_3216Metric_Pad1.42x1.75mm_HandSolder -> Fuse:Fuse_1206_3216Metric; LCSC (none) -> C70069
- FB1: footprint Inductor_SMD:L_0805_2012Metric_Pad1.15x1.40mm_HandSolder -> Inductor_SMD:L_0805_2012Metric; LCSC (none) -> C18305
- R1, R4: footprint Resistor_SMD:R_0805_2012Metric_Pad1.15x1.40mm_HandSolder -> Resistor_SMD:R_0805_2012Metric; LCSC (none) -> C84376
- R2, R3: footprint Resistor_SMD:R_0805_2012Metric_Pad1.15x1.40mm_HandSolder -> Resistor_SMD:R_0805_2012Metric; LCSC (none) -> C150390
- R5, R6: footprint Resistor_SMD:R_0805_2012Metric_Pad1.15x1.40mm_HandSolder -> Resistor_SMD:R_0805_2012Metric; LCSC (none) -> C134293
- U1: LCSC (none) -> C44854
- U2: LCSC (none) -> C12333
- USB1: footprint Type-C:HRO-TYPE-C-31-M-12-HandSoldering -> Type-C:HRO-TYPE-C-31-M-12; LCSC (none) -> C165948
- X1: footprint Crystal:Crystal_SMD_3225-4Pin_3.2x2.5mm_HandSoldering -> Crystal:Crystal_SMD_3225-4Pin_3.2x2.5mm
Changed lines of the file:
@@
 F 2 "Package_QFP:TQFP-44_10x10mm_P0.8mm" H 2900 3350 50  0001 C CIN
 F 3 "http://ww1.microchip.com/downloads/en/DeviceDoc/Atmel-7766-8-bit-AVR-ATmega16U4-32U4_Datasheet.pdf" H 2900 3350 50  0001 C CNN
+F 4 "C44854" H 2900 3350 50  0001 C CNN "LCSC"
 	1    2900 3350
 	1    0    0    -1
@@
 F 0 "R4" V 3904 3950 50  0000 C CNN
 F 1 "10k" V 3995 3950 50  0000 C CNN
-F 2 "Resistor_SMD:R_0805_2012Metric_Pad1.15x1.40mm_HandSolder" H 4100 3950 50  0001 C CNN
+F 2 "Resistor_SMD:R_0805_2012Metric" H 4100 3950 50  0001 C CNN
 F 3 "~" H 4100 3950 50  0001 C CNN
+F 4 "C84376" H 4100 3950 50  0001 C CNN "LCSC"
 	1    4100 3950
 	0    1    1    0
@@
 F 0 "X1" H 1300 4800 50  0000 L CNN
 F 1 "XTAL" H 1500 4500 50  0000 L CNN
-F 2 "Crystal:Crystal_SMD_3225-4Pin_3.2x2.5mm_HandSoldering" H 1450 4650 50  0001 C CNN
+F 2 "Crystal:Crystal_SMD_3225-4Pin_3.2x2.5mm" H 1450 4650 50  0001 C CNN
 F 3 "~" H 1450 4650 50  0001 C CNN
 	1    1450 4650
@@
 F 0 "C1" H 3250 1250 50  0000 L CNN
 F 1 "0.1u" H 3200 1050 50  0000 L CNN
-F 2 "Capacitor_SMD:C_0805_2012Metric_Pad1.15x1.40mm_HandSolder" H 3400 1150 50  0001 C CNN
+F 2 "Capacitor_SMD:C_0805_2012Metric" H 3400 1150 50  0001 C CNN
 F 3 "~" H 3400 1150 50  0001 C CNN
+F 4 "C62912" H 3400 1150 50  0001 C CNN "LCSC"
 	1    3400 1150
 	1    0    0    -1
@@
 F 0 "C2" H 3600 1250 50  0000 L CNN
 F 1 "0.1u" H 3550 1050 50  0000 L CNN
-F 2 "Capacitor_SMD:C_0805_2012Metric_Pad1.15x1.40mm_HandSolder" H 3750 1150 50  0001 C CNN
+F 2 "Capacitor_SMD:C_0805_2012Metric" H 3750 1150 50  0001 C CNN
 F 3 "~" H 3750 1150 50  0001 C CNN
+F 4 "C62912" H 3750 1150 50  0001 C CNN "LCSC"
 	1    3750 1150
 	1    0    0    -1
@@
 F 0 "R1" V 1654 1600 50  0000 C CNN
 F 1 "10k" V 1745 1600 50  0000 C CNN
-F 2 "Resistor_SMD:R_0805_2012Metric_Pad1.15x1.40mm_HandSolder" H 1850 1600 50  0001 C CNN
+F 2 "Resistor_SMD:R_0805_2012Metric" H 1850 1600 50  0001 C CNN
 F 3 "~" H 1850 1600 50  0001 C CNN
+F 4 "C84376" H 1850 1600 50  0001 C CNN "LCSC"
 	1    1850 1600
 	0    1    1    0
@@
 F 0 "R2" V 1750 2850 50  0000 C CNN
 F 1 "22" V 1645 2850 50  0000 C CNN
-F 2 "Resistor_SMD:R_0805_2012Metric_Pad1.15x1.40mm_HandSolder" H 1750 2850 50  0001 C CNN
+F 2 "Resistor_SMD:R_0805_2012Metric" H 1750 2850 50  0001 C CNN
 F 3 "~" H 1750 2850 50  0001 C CNN
+F 4 "C150390" H 1750 2850 50  0001 C CNN "LCSC"
 	1    1750 2850
 	0    1    1    0
@@
 F 0 "R3" V 1750 2950 50  0000 C CNN
 F 1 "22" V 1850 2950 50  0000 C CNN
-F 2 "Resistor_SMD:R_0805_2012Metric_Pad1.15x1.40mm_HandSolder" H 1750 2950 50  0001 C CNN
+F 2 "Resistor_SMD:R_0805_2012Metric" H 1750 2950 50  0001 C CNN
 F 3 "~" H 1750 2950 50  0001 C CNN
+F 4 "C150390" H 1750 2950 50  0001 C CNN "LCSC"
 	1    1750 2950
 	0    1    1    0
@@
 F 0 "USB1" H 6583 2947 60  0000 C CNN
 F 1 "HRO-TYPE-C-31-M-12" H 6583 2841 60  0000 C CNN
-F 2 "Type-C:HRO-TYPE-C-31-M-12-HandSoldering" H 6750 2150 60  0001 C CNN
+F 2 "Type-C:HRO-TYPE-C-31-M-12" H 6750 2150 60  0001 C CNN
 F 3 "" H 6750 2150 60  0001 C CNN
+F 4 "C165948" H 6750 2150 50  0001 C CNN "LCSC"
 	1    6750 2150
 	1    0    0    -1
@@
 F 0 "F1" V 7545 1700 50  0000 C CNN
 F 1 "500" V 7636 1700 50  0000 C CNN
-F 2 "Fuse:Fuse_1206_3216Metric_Pad1.42x1.75mm_HandSolder" H 7800 1500 50  0001 L CNN
+F 2 "Fuse:Fuse_1206_3216Metric" H 7800 1500 50  0001 L CNN
 F 3 "~" H 7750 1700 50  0001 C CNN
+F 4 "C70069" H 7750 1700 50  0001 C CNN "LCSC"
 	1    7750 1700
 	0    1    1    0
@@
 F 0 "R5" V 7250 2500 50  0000 C CNN
 F 1 "5.1k" V 7145 2500 50  0000 C CNN
-F 2 "Resistor_SMD:R_0805_2012Metric_Pad1.15x1.40mm_HandSolder" H 7250 2500 50  0001 C CNN
+F 2 "Resistor_SMD:R_0805_2012Metric" H 7250 2500 50  0001 C CNN
 F 3 "~" H 7250 2500 50  0001 C CNN
+F 4 "C134293" H 7250 2500 50  0001 C CNN "LCSC"
 	1    7250 2500
 	0    1    1    0
@@
 F 0 "R6" H 7400 2450 50  0000 C CNN
 F 1 "5.1k" H 7400 2550 50  0000 C CNN
-F 2 "Resistor_SMD:R_0805_2012Metric_Pad1.15x1.40mm_HandSolder" H 7550 2500 50  0001 C CNN
+F 2 "Resistor_SMD:R_0805_2012Metric" H 7550 2500 50  0001 C CNN
 F 3 "~" H 7550 2500 50  0001 C CNN
+F 4 "C134293" H 7550 2500 50  0001 C CNN "LCSC"
 	1    7550 2500
 	-1   0    0    1
@@
 F 2 "random-keyboard-parts:SOT143B" H 8250 2650 60  0001 C CNN
 F 3 "" H 8250 2650 60  0001 C CNN
+F 4 "C12333" H 8250 2650 50  0001 C CNN "LCSC"
 	1    8250 2650
 	1    0    0    -1
@@
 F 0 "C8" H 1992 4846 50  0000 L CNN
 F 1 "22p" H 1992 4755 50  0000 L CNN
-F 2 "Capacitor_SMD:C_0805_2012Metric_Pad1.15x1.40mm_HandSolder" H 1900 4800 50  0001 C CNN
+F 2 "Capacitor_SMD:C_0805_2012Metric" H 1900 4800 50  0001 C CNN
 F 3 "~" H 1900 4800 50  0001 C CNN
+F 4 "C1804" H 1900 4800 50  0001 C CNN "LCSC"
 	1    1900 4800
 	1    0    0    -1
@@
 F 0 "C7" H 900 4850 50  0000 L CNN
 F 1 "22p" H 900 4750 50  0000 L CNN
-F 2 "Capacitor_SMD:C_0805_2012Metric_Pad1.15x1.40mm_HandSolder" H 1150 4800 50  0001 C CNN
+F 2 "Capacitor_SMD:C_0805_2012Metric" H 1150 4800 50  0001 C CNN
 F 3 "~" H 1150 4800 50  0001 C CNN
+F 4 "C1804" H 1150 4800 50  0001 C CNN "LCSC"
 	1    1150 4800
 	1    0    0    -1
@@
 F 0 "C6" H 1992 3446 50  0000 L CNN
 F 1 "1u" H 1992 3355 50  0000 L CNN
-F 2 "Capacitor_SMD:C_0805_2012Metric_Pad1.15x1.40mm_HandSolder" H 1900 3400 50  0001 C CNN
+F 2 "Capacitor_SMD:C_0805_2012Metric" H 1900 3400 50  0001 C CNN
 F 3 "~" H 1900 3400 50  0001 C CNN
+F 4 "C116352" H 1900 3400 50  0001 C CNN "LCSC"
 	1    1900 3400
 	1    0    0    -1
@@
 F 0 "C5" H 4300 1250 50  0000 L CNN
 F 1 "10u" H 4250 1050 50  0000 L CNN
-F 2 "Capacitor_SMD:C_0805_2012Metric_Pad1.15x1.40mm_HandSolder" H 4450 1150 50  0001 C CNN
+F 2 "Capacitor_SMD:C_0805_2012Metric" H 4450 1150 50  0001 C CNN
 F 3 "~" H 4450 1150 50  0001 C CNN
+F 4 "C95841" H 4450 1150 50  0001 C CNN "LCSC"
 	1    4450 1150
 	1    0    0    -1
@@
 F 0 "C3" H 3950 1250 50  0000 L CNN
 F 1 "0.1u" H 3900 1050 50  0000 L CNN
-F 2 "Capacitor_SMD:C_0805_2012Metric_Pad1.15x1.40mm_HandSolder" H 4100 1150 50  0001 C CNN
+F 2 "Capacitor_SMD:C_0805_2012Metric" H 4100 1150 50  0001 C CNN
 F 3 "~" H 4100 1150 50  0001 C CNN
-F 4 "" H 4100 1150 50  0001 C CNN "LCSC"
+F 4 "C62912" H 4100 1150 50  0001 C CNN "LCSC"
 	1    4100 1150
 	1    0    0    -1
@@
 F 0 "FB1" V 6263 3200 50  0000 C CNN
 F 1 "60@100Mhz" V 6354 3200 50  0000 C CNN
-F 2 "Inductor_SMD:L_0805_2012Metric_Pad1.15x1.40mm_HandSolder" V 6430 3200 50  0001 C CNN
+F 2 "Inductor_SMD:L_0805_2012Metric" V 6430 3200 50  0001 C CNN
 F 3 "~" H 6500 3200 50  0001 C CNN
+F 4 "C18305" H 6500 3200 50  0001 C CNN "LCSC"
 	1    6500 3200
 	0    1    1    0
