File: PCB/CrowMiniMk2.kicad_pcb (KiCad board)
At the start: 2 copper layers, 316.7 x 100.6 mm, 36 parts, among them K42 ', K43 ENTER, K44 LSHIFT, K45 Z, K46 X, K47 C, K48 V, K49 B, K50 N, K51 M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

Commit message: Some routing done
Parts:
- added K8: #7, MX_Only:MXOnly-1U-NoLED, F.Cu at (152.4, 44.5)
- moved R2 4.20 mm to (155.4, 106.7), turned to 180 degrees
- moved X1 2.87 mm to (174.9, 120.0), turned to 90 degrees
- moved R3 1.36 mm to (155.4, 109.0), turned to 180 degrees
- moved R6 0.77 mm to (25.4, 42.1)
- moved U2 0.13 mm to (28.4, 47.8)
Routing:
- net ROW0: track 0.00 -> 315.8 mm, vias 0 -> 2
- net ROW4: track 0.00 -> 303.2 mm
- net ROW1: track 0.00 -> 292.9 mm, vias 0 -> 2
- net ROW3: track 0.00 -> 264.4 mm, vias 0 -> 2
- net ROW2: track 0.00 -> 251.7 mm, vias 0 -> 2
- net D+: track 0.00 -> 211.2 mm
- net D-: track 0.00 -> 210.2 mm
- net COL12: track 0.00 -> 108.0 mm
- net COL11: track 0.00 -> 104.2 mm
- net COL10: track 0.00 -> 100.1 mm
- net COL9: track 0.00 -> 95.9 mm
- net COL0: track 0.00 -> 94.2 mm
- net COL6: track 0.00 -> 92.4 mm
- net COL2: track 0.00 -> 91.9 mm
- net COL1: track 0.00 -> 84.2 mm
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Other:
- board size 316.7 x 100.6 mm -> 317.2 x 100.8 mm

Commit message: Routing 99%
Parts:
- added C5: 10u, Capacitor_SMD:C_0805_2012Metric_Pad1.15x1.40mm_HandSolder, B.Cu at (151.4, 112.0)
- added C6: 1u, Capacitor_SMD:C_0805_2012Metric_Pad1.15x1.40mm_HandSolder, B.Cu at (161.8, 107.7)
- moved R1 11.9 mm to (106.2, 122.7)
- moved SW1 4.35 mm to (99.1, 120.9), turned to 180 degrees
- moved R4 0.76 mm to (152.1, 127.8)
Connections:
- U1 pad 38: ROW1 -> ROW4
- U1 pad 39: ROW4 -> ROW3
- U1 pad 40: ROW3 -> ROW2
- U1 pad 41: ROW2 -> ROW1
Routing:
- net +5V: track 8.88 -> 351.1 mm, vias 0 -> 17
- net GND: track 30.5 -> 358.2 mm, vias 0 -> 10
- net COL0: track 94.2 -> 262.0 mm, vias 0 -> 1
- net COL14: track 77.5 -> 239.1 mm, vias 0 -> 1
- net COL13: track 76.7 -> 236.0 mm, vias 0 -> 1
- net COL1: track 84.2 -> 230.1 mm, vias 0 -> 1
- net COL2: track 91.9 -> 217.4 mm, vias 0 -> 1
- net COL12: track 108.0 -> 227.3 mm, vias 0 -> 1
- net COL4: track 71.9 -> 186.3 mm, vias 0 -> 1
- net COL3: track 73.2 -> 183.3 mm, vias 0 -> 1
- net RST: track 0.00 -> 101.3 mm, vias 0 -> 5
- net COL11: track 104.2 -> 198.8 mm, vias 0 -> 3
- net ROW0: track 315.8 -> 405.7 mm, vias 2 -> 8
- net MOSI: track 0.00 -> 78.6 mm, vias 0 -> 6
- net MISO: track 0.00 -> 72.4 mm, vias 0 -> 8
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
Commit message: Pre Logo add
Parts:
- removed C5: 10u, Capacitor_SMD:C_0805_2012Metric_Pad1.15x1.40mm_HandSolder
- removed C6: 1u, Capacitor_SMD:C_0805_2012Metric_Pad1.15x1.40mm_HandSolder
- removed K8: #7, MX_Only:MXOnly-1U-NoLED
- removed R1, R4: 10k, Resistor_SMD:R_0805_2012Metric_Pad1.15x1.40mm_HandSolder
- removed R2, R3: 22, Resistor_SMD:R_0805_2012Metric_Pad1.15x1.40mm_HandSolder
- removed R5, R6: 5.1k, Resistor_SMD:R_0805_2012Metric_Pad1.15x1.40mm_HandSolder
- removed SW1: SW_Push, Button_Switch_SMD:SW_SPST_SKQG_WithStem
- removed U1: ATmega32U4-AU, Package_QFP:TQFP-44_10x10mm_P0.8mm
- removed U2: PRTR5V0U2X, random-keyboard-parts:SOT143B
- removed USB1: HRO-TYPE-C-31-M-12, Type-C:HRO-TYPE-C-31-M-12-HandSoldering
- removed X1: XTAL, Crystal:Crystal_SMD_3225-4Pin_3.2x2.5mm_HandSoldering
- added K14: BACK, local:MXOnly-2U-NoLED, F.Cu at (276.2, 44.5)
- added K16: TAB, local:MXOnly-1.5U-NoLED, F.Cu at (23.8, 63.5)
- added K29: \|, local:MXOnly-1.5U-NoLED, F.Cu at (281.0, 63.5)
- added K31: CAPSLOCK, local:MXOnly-1.75U-NoLED, F.Cu at (26.2, 82.5)
- K42, K45, K46, K47, K48, K49, K50, K51, K52, K53, K54, K56, K58, K64, K65, K66: footprint MX_Only:MXOnly-1U-NoLED -> local:MXOnly-1U-NoLED
- K43, K44, K55: footprint MX_Only:MXOnly-2.25U-NoLED -> local:MXOnly-2.25U-NoLED
- K57, K59, K61, K62, K63: footprint MX_Only:MXOnly-1.25U-NoLED -> local:MXOnly-1.25U-NoLED
- K60: footprint MX_Only:MXOnly-6.25U-NoLED -> local:MXOnly-6.25U-NoLED
Routing:
- net Earth: track 0.00 -> 20.2 mm
- net GND: track 358.2 -> 370.0 mm, vias 10 -> 15
- added copper zone on B.Cu, net GND
- added copper zone on F.Cu, net GND
